Commit message: Added yaml file for xacro properties. Seems right. (Task A.3)
diff_params.yaml:
+ Created

turtlebot3_burger.urdf.xacro:
+ Now reads wheel_radius, track_width, collision_radius from diff_params

Next steps:
Add color namespaces (Task A.4)

File: nuturtle_description/urdf/turtlebot3_burger.urdf.xacro (robot description, xacro)
@@ -1,6 +1,12 @@
 <?xml version="1.0" ?>
+<!-- Test comment  -->
 <robot name="turtlebot3_burger" xmlns:xacro="http://ros.org/wiki/xacro">
   <xacro:arg name="namespace" default=""/>
   <xacro:property name="namespace" value="$(arg namespace)"/>
+  <xacro:property name="property_yaml" value="$(find nuturtle_description)/config/diff_params.yaml" />
+  <xacro:property name="main_props" value="${xacro.load_yaml(property_yaml)['/**']['ros__parameters']}" />
+  <xacro:property name="wheel_radius"  value="${main_props['wheel_radius']}" />
+  <xacro:property name="track_width"  value="${main_props['track_width']}" />
+  <xacro:property name="collision_radius"  value="${main_props['collision_radius']}" />
   <!-- Init colour -->
   <material name="black">
@@ -48,8 +54,14 @@
       <material name="light_black"/>
     </visual>
+    <!-- <collision>
+      <origin xyz="-0.032 0 0.070" rpy="0 0 0"/>
+      <geometry>
+        <box size="0.140 0.140 0.143"/>
+      </geometry>
+    </collision> -->
     <collision>
       <origin xyz="-0.032 0 0.070" rpy="0 0 0"/>
       <geometry>
-        <box size="0.140 0.140 0.143"/>
+        <cylinder length="0.143" radius="${collision_radius}" />
       </geometry>
     </collision>
@@ -63,5 +75,5 @@
     <parent link="${namespace}base_link"/>
     <child link="${namespace}wheel_left_link"/>
-    <origin xyz="0.0 0.08 0.023" rpy="-1.57 0 0"/>
+    <origin xyz="0.0 ${track_width/2} 0.023" rpy="-1.57 0 0"/>
     <axis xyz="0 0 1"/>
   </joint>
@@ -77,5 +89,5 @@
       <origin xyz="0 0 0" rpy="0 0 0"/>
       <geometry>
-        <cylinder length="0.018" radius="0.033"/>
+        <cylinder length="0.018" radius="${wheel_radius}"/>
       </geometry>
     </collision>
@@ -89,5 +101,5 @@
     <parent link="${namespace}base_link"/>
     <child link="${namespace}wheel_right_link"/>
-    <origin xyz="0.0 -0.080 0.023" rpy="-1.57 0 0"/>
+    <origin xyz="0.0 ${-track_width/2} 0.023" rpy="-1.57 0 0"/>
     <axis xyz="0 0 1"/>
   </joint>
@@ -103,5 +115,5 @@
       <origin xyz="0 0 0" rpy="0 0 0"/>
       <geometry>
-        <cylinder length="0.018" radius="0.033"/>
+        <cylinder length="0.018" radius="${wheel_radius}"/>
       </geometry>
     </collision>

Commit message: Added color argument xacro and launchfile (Task A.4)
load_one.launch.xml:
+  Added arg `color` that gets passed into the xacro and is used for
++ all node namespaces. Values restricted to red, blue, green, purple.
+  robot_state_publisher frame_prefix is set to the value of `color`.
+  Args `use_rviz` and `use_jsp` now take bools instead of strings.

turtlebot3_burger.urdf.xacro:
+  Added `color` argument that changes the color of the base_links.

Added rviz configs for colors.
load_one_`color`.rviz (4 separate files):
+  Fixed frame is set to `color`/base_link.
+  RobotModel TF prefix is set to `color`
+  RobotModel topic is set to `color`/robot_description

Next steps:
Task A.5 (load_all.launch.xml)
Figure out xacro comments
Get launchfiles to properly close everything when rviz is closed

File: nuturtle_description/urdf/turtlebot3_burger.urdf.xacro (robot description, xacro)
@@ -2,4 +2,6 @@
 <!-- Test comment  -->
 <robot name="turtlebot3_burger" xmlns:xacro="http://ros.org/wiki/xacro">
+  <xacro:arg name="color" default=""/>
+  <xacro:property name="color" value="$(arg color)"/>
   <xacro:arg name="namespace" default=""/>
   <xacro:property name="namespace" value="$(arg namespace)"/>
@@ -10,4 +12,7 @@
   <xacro:property name="collision_radius"  value="${main_props['collision_radius']}" />
   <!-- Init colour -->
+  <material name="purple">
+      <color rgba="0.3 0.16 0.52 1.0"/>
+  </material>
   <material name="black">
       <color rgba="0.0 0.0 0.0 1.0"/>
@@ -52,5 +57,5 @@
         <mesh filename="package://nuturtle_description/meshes/burger_base.stl" scale="0.001 0.001 0.001"/>
       </geometry>
-      <material name="light_black"/>
+      <material name="${color}"/>
     </visual>
     <!-- <collision>
